File: SDR_STM32L0_1.2/KicadFiles/Peripheral.kicad_sch (KiCad schematic)
At the start: 22 parts, among them J1 Conn_01x03, J2 USB_C_Receptacle_USB2.0_16P, P1 3220-20-0200-00, SW2 RESET SWITCH, U2 Engine-Controller_SST25VF040B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, U5 CP2102N-Axx-xQFN28

Commit message: dev
Connections:
- net FLASH_SELECT renamed SPI1_NSS
Changed lines of the file:
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@@
 		)
 	)
-	(global_label "FLASH_SELECT"
+	(global_label "SPI1_NSS"
 		(shape input)
 		(at 199.39 31.75 180)
@@
 		)
 		(property "Intersheetrefs" "${INTERSHEET_REFS}"
-			(at 182.9187 31.75 0)
+			(at 187.3939 31.75 0)
 			(effects
 				(font

Commit message: added 1.2 back
Parts:
- P1: footprint USBs:3220-20-0200-00 -> Connector_USB:3220-20-0200-00
- U2: footprint USBs:SST25VF040B-50-4I-S2AE-T -> Connector_USB:SST25VF040B-50-4I-S2AE-T
Connections:
- net SPI1_NSS renamed FLASH_SELECT
Changed lines of the file:
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@@
 		)
 	)
-	(global_label "SPI1_NSS"
+	(global_label "FLASH_SELECT"
 		(shape input)
 		(at 199.39 31.75 180)
@@
 		)
 		(property "Intersheetrefs" "${INTERSHEET_REFS}"
-			(at 187.3939 31.75 0)
+			(at 182.9187 31.75 0)
 			(effects
 				(font
@@
 			)
 		)
-		(property "Footprint" "USBs:3220-20-0200-00"
+		(property "Footprint" "Connector_USB:3220-20-0200-00"
 			(at 54.61 136.144 0)
 			(effects
@@
 			)
 		)
-		(property "Footprint" "USBs:SST25VF040B-50-4I-S2AE-T"
+		(property "Footprint" "Connector_USB:SST25VF040B-50-4I-S2AE-T"
 			(at 218.44 52.07 0)
 			(effects
